Commit message: Follow simple.js example

File: examples/niryo_simple.urdf (robot description, URDF)
Before this commit: robot simple_niryo, 13 links, 12 joints
Links:
- removed link left_finger_link
- removed link right_finger_link
Joints:
- removed joint knuckle_to_left_finger_joint
- removed joint knuckle_to_right_finger_joint
