Commit message: Change endpoint to ros/pkgs and add examples

File: examples/niryo.urdf (robot description, URDF)
Before this commit: robot simple_niryo, 13 links, 12 joints
Joints:
- joint base_to_shoulder_joint: limit lower=-${radians(150.0)} upper=${radians(150.0)} effort=1000.0 velocity=0.5 -> lower=-2.617994 upper=2.617994 effort=1000.0 velocity=0.5
- joint elbow_to_wrist_joint: limit lower=${radians(-100.0)} upper=${radians(100.0)} effort=1000.0 velocity=0.5 -> lower=-1.745329 upper=1.745329 effort=1000.0 velocity=0.5
- joint shoulder_to_elbow_joint: limit lower=${radians(-10.0)} upper=${radians(200.0)} effort=1000.0 velocity=0.5 -> lower=-0.1745329 upper=3.490659 effort=1000.0 velocity=0.5; origin xyz=0 0 0.15 rpy=${radians(90)} 0 0 -> xyz=0 0 0.15 rpy=1.570796 0 0
- joint wrist_to_hand_joint: limit lower=${radians(-90.0)} upper=${radians(90.0)} effort=1000.0 velocity=0.5 -> lower=-1.570796 upper=1.570796 effort=1000.0 velocity=0.5
