Commit message: Add examples and rename packages

File: examples/T12_flipped.urdf (robot description, URDF)
Before this commit: robot T12, 37 links, 36 joints
Links:
- link Ankle1: geometry collision mesh filename=package://t12_description/meshes/Ankle1.STL; visual mesh filename=package://t12_description/meshes/Ankle1.STL
- link Ankle2: geometry collision mesh filename=package://t12_description/meshes/Ankle2.STL; visual mesh filename=package://t12_description/meshes/Ankle2.STL
- link Ankle3: geometry collision mesh filename=package://t12_description/meshes/Ankle3.STL; visual mesh filename=package://t12_description/meshes/Ankle3.STL
- link Ankle4: geometry collision mesh filename=package://t12_description/meshes/Ankle4.STL; visual mesh filename=package://t12_description/meshes/Ankle4.STL
- link Ankle5: geometry collision mesh filename=package://t12_description/meshes/Ankle5.STL; visual mesh filename=package://t12_description/meshes/Ankle5.STL
- link Ankle6: geometry collision mesh filename=package://t12_description/meshes/Ankle6.STL; visual mesh filename=package://t12_description/meshes/Ankle6.STL
- link Body: geometry collision mesh filename=package://t12_description/meshes/Body.STL; visual mesh filename=package://t12_description/meshes/Body.STL
- link Foot1: geometry collision mesh filename=package://t12_description/meshes/Foot1.STL; visual mesh filename=package://t12_description/meshes/Foot1.STL
- link Foot2: geometry collision mesh filename=package://t12_description/meshes/Foot2.STL; visual mesh filename=package://t12_description/meshes/Foot2.STL
- link Foot3: geometry collision mesh filename=package://t12_description/meshes/Foot3.STL; visual mesh filename=package://t12_description/meshes/Foot3.STL
- link Foot4: geometry collision mesh filename=package://t12_description/meshes/Foot4.STL; visual mesh filename=package://t12_description/meshes/Foot4.STL
- link Foot5: geometry collision mesh filename=package://t12_description/meshes/Foot5.STL; visual mesh filename=package://t12_description/meshes/Foot5.STL
- link Foot6: geometry collision mesh filename=package://t12_description/meshes/Foot6.STL; visual mesh filename=package://t12_description/meshes/Foot6.STL
- link Hip1: geometry collision mesh filename=package://t12_description/meshes/Hip1.STL; visual mesh filename=package://t12_description/meshes/Hip1.STL
- link Hip2: geometry collision mesh filename=package://t12_description/meshes/Hip2.STL; visual mesh filename=package://t12_description/meshes/Hip2.STL
- link Hip3: geometry collision mesh filename=package://t12_description/meshes/Hip3.STL; visual mesh filename=package://t12_description/meshes/Hip3.STL
- link Hip4: geometry collision mesh filename=package://t12_description/meshes/Hip4.STL; visual mesh filename=package://t12_description/meshes/Hip4.STL
- link Hip5: geometry collision mesh filename=package://t12_description/meshes/Hip5.STL; visual mesh filename=package://t12_description/meshes/Hip5.STL
- link Hip6: geometry collision mesh filename=package://t12_description/meshes/Hip6.STL; visual mesh filename=package://t12_description/meshes/Hip6.STL
- link Knee1: geometry collision mesh filename=package://t12_description/meshes/Knee1.STL; visual mesh filename=package://t12_description/meshes/Knee1.STL
- link Knee2: geometry collision mesh filename=package://t12_description/meshes/Knee2.STL; visual mesh filename=package://t12_description/meshes/Knee2.STL
- link Knee3: geometry collision mesh filename=package://t12_description/meshes/Knee3.STL; visual mesh filename=package://t12_description/meshes/Knee3.STL
- link Knee4: geometry collision mesh filename=package://t12_description/meshes/Knee4.STL; visual mesh filename=package://t12_description/meshes/Knee4.STL
- link Knee5: geometry collision mesh filename=package://t12_description/meshes/Knee5.STL; visual mesh filename=package://t12_description/meshes/Knee5.STL
- link Knee6: geometry collision mesh filename=package://t12_description/meshes/Knee6.STL; visual mesh filename=package://t12_description/meshes/Knee6.STL
- link Shin1: geometry collision mesh filename=package://t12_description/meshes/Shin1.STL; visual mesh filename=package://t12_description/meshes/Shin1.STL
- link Shin2: geometry collision mesh filename=package://t12_description/meshes/Shin2.STL; visual mesh filename=package://t12_description/meshes/Shin2.STL
- link Shin3: geometry collision mesh filename=package://t12_description/meshes/Shin3.STL; visual mesh filename=package://t12_description/meshes/Shin3.STL
- link Shin4: geometry collision mesh filename=package://t12_description/meshes/Shin4.STL; visual mesh filename=package://t12_description/meshes/Shin4.STL
- link Shin5: geometry collision mesh filename=package://t12_description/meshes/Shin5.STL; visual mesh filename=package://t12_description/meshes/Shin5.STL
- link Shin6: geometry collision mesh filename=package://t12_description/meshes/Shin6.STL; visual mesh filename=package://t12_description/meshes/Shin6.STL
- link Thigh1: geometry collision mesh filename=package://t12_description/meshes/Thigh1.STL; visual mesh filename=package://t12_description/meshes/Thigh1.STL
- link Thigh2: geometry collision mesh filename=package://t12_description/meshes/Thigh2.STL; visual mesh filename=package://t12_description/meshes/Thigh2.STL
- link Thigh3: geometry collision mesh filename=package://t12_description/meshes/Thigh3.STL; visual mesh filename=package://t12_description/meshes/Thigh3.STL
- link Thigh4: geometry collision mesh filename=package://t12_description/meshes/Thigh4.STL; visual mesh filename=package://t12_description/meshes/Thigh4.STL
- link Thigh5: geometry collision mesh filename=package://t12_description/meshes/Thigh5.STL; visual mesh filename=package://t12_description/meshes/Thigh5.STL
- link Thigh6: geometry collision mesh filename=package://t12_description/meshes/Thigh6.STL; visual mesh filename=package://t12_description/meshes/Thigh6.STL

File: examples/spot.urdf (robot description, URDF)
Before this commit: robot spot, 13 links, 12 joints
Links:
- link base: geometry visual mesh filename=package://spot_description/meshes/base.stl
- link fl.hip: geometry visual mesh filename=package://spot_description/meshes/fl.hip.stl
- link fl.lleg: geometry visual mesh filename=package://spot_description/meshes/fl.lleg.stl
- link fl.uleg: geometry visual mesh filename=package://spot_description/meshes/fl.uleg.stl
- link fr.hip: geometry visual mesh filename=package://spot_description/meshes/fr.hip.stl
- link fr.lleg: geometry visual mesh filename=package://spot_description/meshes/fr.lleg.stl
- link fr.uleg: geometry visual mesh filename=package://spot_description/meshes/fr.uleg.stl
- link hl.hip: geometry visual mesh filename=package://spot_description/meshes/hl.hip.stl
- link hl.lleg: geometry visual mesh filename=package://spot_description/meshes/hl.lleg.stl
- link hl.uleg: geometry visual mesh filename=package://spot_description/meshes/hl.uleg.stl
- link hr.hip: geometry visual mesh filename=package://spot_description/meshes/hr.hip.stl
- link hr.lleg: geometry visual mesh filename=package://spot_description/meshes/hr.lleg.stl
- link hr.uleg: geometry visual mesh filename=package://spot_description/meshes/hr.uleg.stl
