Commit message: Add prismatic joint example

File: examples/basic.urdf (robot description, URDF)
Before this commit: robot myfirst, 1 links, 0 joints
Links:
- added link plate; visual box size=0.7 0.7 0.05
- link base_link: geometry visual cylinder length=1 radius=0.25
Joints:
- added joint base_to_plate: type prismatic, parent base_link, child plate, origin xyz=0 0 0 rpy=0 0 0, axis 0 0 1, limit lower=0 upper=1 effort=1000.0 velocity=0.5
