Commit message: Add examples and improve mesh path parsing

File: examples/racecar/racecar.urdf (robot description, URDF)
Before this commit: robot racecar, 13 links, 12 joints
Links:
- link chassis: geometry visual mesh filename=meshes/chassis.STL
- link laser: geometry collision box size=0.1 0.1 0.1; visual mesh filename=meshes/hokuyo.obj
- link left_front_wheel: geometry collision cylinder length=0.045 radius=0.05; visual mesh filename=meshes/left_front_wheel.obj
- link left_rear_wheel: geometry collision cylinder length=0.045 radius=0.05; visual mesh filename=meshes/left_rear_wheel.obj
- link left_steering_hinge: geometry visual mesh filename=meshes/left_steering_hinge.STL
- link right_front_wheel: geometry collision cylinder length=0.045 radius=0.05; visual mesh filename=meshes/right_front_wheel.obj
- link right_rear_wheel: geometry collision cylinder length=0.045 radius=0.05; visual mesh filename=meshes/right_rear_wheel.obj
- link right_steering_hinge: geometry visual mesh filename=meshes/right_steering_hinge.STL
